Commit message: both end-effectors work with a single launch file

File: config/srdf/ur.srdf.xacro (robot description, xacro)
@@ -16,3 +16,11 @@
     <xacro:ur_nailgun_srdf />
   </xacro:if>
+  <xacro:if value="${'$(arg end_effector_type)' == 'both'}">
+    <xacro:ur_simple_gripper_srdf />
+    <xacro:ur_nailgun_srdf />
+    <!-- Cross-collisions between gripper and nailgun -->
+    <disable_collisions link1="gripper_base" link2="nailgun_base" reason="Never" />
+    <disable_collisions link1="gripper_left_finger" link2="nailgun_base" reason="Never" />
+    <disable_collisions link1="gripper_right_finger" link2="nailgun_base" reason="Never" />
+  </xacro:if>
 </robot>

File: config/srdf/ur_nailgun_macro.srdf.xacro (robot description, xacro)
@@ -10,4 +10,5 @@
     <!-- Disable collisions for nailgun -->
     <disable_collisions link1="nailgun_base" link2="tool0" reason="Adjacent" />
+    <disable_collisions link1="nailgun_base" link2="flange" reason="Adjacent" />
     <disable_collisions link1="nailgun_base" link2="wrist_3_link" reason="Never" />
     <disable_collisions link1="nailgun_base" link2="wrist_2_link" reason="Never" />

File: urdf/ur.urdf.xacro (robot description, xacro)
@@ -14,5 +14,5 @@
    <xacro:arg name="tf_prefix" default="" />
    <xacro:arg name="joint_limit_params" default="$(find ur_description)/config/$(arg ur_type)/joint_limits.yaml"/>
-   <xacro:arg name="kinematics_params" default="$(find ur_description)/config/$(arg ur_type)/default_kinematics.yaml"/>
+   <xacro:arg name="kinematics_params" default="$(find hello_moveit)/config/robot_calibration.yaml"/>
    <xacro:arg name="physical_params" default="$(find ur_description)/config/$(arg ur_type)/physical_parameters.yaml"/>
    <xacro:arg name="visual_params" default="$(find ur_description)/config/$(arg ur_type)/visual_parameters.yaml"/>
@@ -45,8 +45,12 @@
    <!-- Conditional instantiation using xacro:if -->
    <xacro:if value="${'$(arg end_effector_type)' == 'gripper'}">
-      <xacro:ur_simple_gripper parent_link="flange" mesh_scale="1 1 1"/>
+      <xacro:ur_simple_gripper parent_link="tool0" mesh_scale="1 1 1"/>
     </xacro:if>
     <xacro:if value="${'$(arg end_effector_type)' == 'nailgun'}">
-      <xacro:ur_nailgun parent_link="flange" mesh_scale="1 1 1"/>
+      <xacro:ur_nailgun parent_link="tool0" mesh_scale="1 1 1"/>
+    </xacro:if>
+    <xacro:if value="${'$(arg end_effector_type)' == 'both'}">
+      <xacro:ur_simple_gripper parent_link="tool0" mesh_scale="1 1 1"/>
+      <xacro:ur_nailgun parent_link="tool0" mesh_scale="1 1 1"/>
     </xacro:if>
    <!-- Add more xacro:if blocks for other end-effectors -->

File: urdf/ur_nailgun.xacro (robot description, xacro)
@@ -1,5 +1,5 @@
 <?xml version="1.0"?>
 <robot xmlns:xacro="http://www.ros.org/wiki/xacro">
-  <xacro:macro name="ur_nailgun" params="parent_link:=flange mesh_scale:='1 1 1'">
+  <xacro:macro name="ur_nailgun" params="parent_link:=tool0 mesh_scale:='1 1 1'">
     <!-- Nailgun base link -->
     <link name="nailgun_base">
@@ -21,5 +21,5 @@
       </inertial>
     </link>
-    <!-- Fixed joint to attach nailgun base to flange -->
+    <!-- Fixed joint to attach nailgun base to tool0 -->
     <joint name="nailgun_base_joint" type="fixed">
       <parent link="${parent_link}"/>
@@ -32,5 +32,5 @@
       <parent link="nailgun_base"/>
       <child link="nailgun_tip"/>
-      <origin xyz="0.268 0.0 0.0" rpy="0 0 0"/>
+      <origin xyz="-0.095 0.0 0.3165" rpy="0 0 0"/>
     </joint>
   </xacro:macro>

File: urdf/ur_simple_gripper.xacro (robot description, xacro)
@@ -1,6 +1,6 @@
 <?xml version="1.0"?>
 <robot xmlns:xacro="http://www.ros.org/wiki/xacro">
-  <!-- Macro for the simple gripper attached to the UR flange -->
-  <xacro:macro name="ur_simple_gripper" params="parent_link:=flange mesh_scale:='1 1 1'">
+  <!-- Macro for the simple gripper attached to the UR tool0 -->
+  <xacro:macro name="ur_simple_gripper" params="parent_link:=tool0 mesh_scale:='1 1 1'">
     <!-- Grippesr base link -->
     <link name="gripper_base">
@@ -18,9 +18,9 @@
   <inertial>
     <mass value="0.425"/>
-    <origin xyz="0.17925 -0.34281 -0.07809" rpy="0 0 0"/>
+    <origin xyz="0.17925 -0.34281 -0.07809" rpy="0 1.5708 0"/>
     <inertia ixx="0.443" ixy="0.0" ixz="0.0" iyy="0.428" iyz="0.0" izz="0.281"/>
   </inertial>
 </link>
-    <!-- Fixed joint to attach gripper base to flange -->
+    <!-- Fixed joint to attach gripper base to tool0 -->
     <joint name="gripper_base_joint" type="fixed">
       <parent link="${parent_link}"/>
@@ -84,9 +84,11 @@
     </joint>
     <!-- Gripper tip link (grasp point between fingertips) -->
+    <!-- gripper_base now has same axes as tool0, so pendant TCP values map directly: -->
+    <!-- pendant X=10mm -> gb X, Y=0 -> gb Y, Z=148mm -> gb Z (outward) -->
     <link name="gripper_tip"/>
     <joint name="gripper_tip_joint" type="fixed">
       <parent link="gripper_base"/>
       <child link="gripper_tip"/>
-      <origin xyz="0.1325 0.0 -0.00735" rpy="0 0 0"/>
+      <origin xyz="0.003 0.0 0.148" rpy="0 0 0"/>
     </joint>
   </xacro:macro>
