Commit message: adjustemnts to measurments

File: urdf/ur_nailgun.xacro (robot description, xacro)
@@ -27,4 +27,11 @@
       <origin xyz="0 0 0" rpy="0 0 0"/>
     </joint>
+    <!-- Nailgun tip link (nozzle point) -->
+    <link name="nailgun_tip"/>
+    <joint name="nailgun_tip_joint" type="fixed">
+      <parent link="nailgun_base"/>
+      <child link="nailgun_tip"/>
+      <origin xyz="0.268 0.0 0.0" rpy="0 0 0"/>
+    </joint>
   </xacro:macro>
 </robot>

File: urdf/ur_simple_gripper.xacro (robot description, xacro)
@@ -83,4 +83,11 @@
       <limit lower="0.0" upper="0.003" effort="10" velocity="0.1"/>
     </joint>
+    <!-- Gripper tip link (grasp point between fingertips) -->
+    <link name="gripper_tip"/>
+    <joint name="gripper_tip_joint" type="fixed">
+      <parent link="gripper_base"/>
+      <child link="gripper_tip"/>
+      <origin xyz="0.1325 0.0 -0.00735" rpy="0 0 0"/>
+    </joint>
   </xacro:macro>
 </robot>

Commit message: final touches

File: urdf/ur_nailgun.xacro (robot description, xacro)
@@ -16,6 +16,6 @@
       </collision>
       <inertial>
-        <mass value="7.3"/>
-        <origin xyz="0.152685 0.098458 -0.00549" rpy="0 0 0"/>
+        <mass value="8.250"/>
+        <origin xyz="-0.013 0.001 0.151" rpy="0 0 0"/>
         <inertia ixx="0.423" ixy="0.0" ixz="0.0" iyy="0.249" iyz="0.0" izz="0.623"/>
       </inertial>
@@ -32,5 +32,5 @@
       <parent link="nailgun_base"/>
       <child link="nailgun_tip"/>
-      <origin xyz="-0.095 0.0 0.3165" rpy="0 0 0"/>
+      <origin xyz="-0.09515 -0.00026 0.3165" rpy="0 0 0"/>
     </joint>
   </xacro:macro>

File: urdf/ur_simple_gripper.xacro (robot description, xacro)
@@ -17,6 +17,6 @@
   </collision>
   <inertial>
-    <mass value="0.425"/>
-    <origin xyz="0.17925 -0.34281 -0.07809" rpy="0 1.5708 0"/>
+    <mass value="0.960"/>
+    <origin xyz="-0.001 0.015 0.028" rpy="0 0 0"/>
     <inertia ixx="0.443" ixy="0.0" ixz="0.0" iyy="0.428" iyz="0.0" izz="0.281"/>
   </inertial>
@@ -42,6 +42,6 @@
   </collision>
   <inertial>
-  <mass value="0.015"/>
-  <origin xyz="0.17913 -0.34967 -0.14886" rpy="0 0 0"/>
+  <mass value="0.0"/>
+  <origin xyz="0 0 0" rpy="0 0 0"/>
   <inertia ixx="0.00131" ixy="0.0" ixz="0.0" iyy="0.00122" iyz="0.0" izz="0.00058"/>
 </inertial>
@@ -70,6 +70,6 @@
   </collision>
   <inertial>
-  <mass value="0.0397"/>
-  <origin xyz="0.17928 -0.31604 -0.15581" rpy="0 0 0"/>
+  <mass value="0.0"/>
+  <origin xyz="0 0 0" rpy="0 0 0"/>
   <inertia ixx="0.0084" ixy="0.0" ixz="0.0" iyy="0.0559" iyz="0.0" izz="0.0494"/>
 </inertial>
@@ -90,5 +90,5 @@
       <parent link="gripper_base"/>
       <child link="gripper_tip"/>
-      <origin xyz="0.003 0.0 0.148" rpy="0 0 0"/>
+      <origin xyz="0.00723 0.00095 0.1465" rpy="0 0 0"/>
     </joint>
   </xacro:macro>
